File: hardware/pcbs/teensy_shield/potentiostat.sch (KiCad schematic (older format))
At the start: 95 parts, among them K1 CONN_3, P1 CONN_2, P10 CONN_2, P11 CONN_2, P12 CONN_2, P13 CONN_5X2, P14 CONN_5X2, P15 CONN_2X2, P16 CONN_2X2, P17 CONN_2, P18 CONN_2, P19 CONN_2, P2 CONN_2, P20 CONN_2, P21 CONN_2, P3 CONN_2, P4 CONN_2, P5 CONN_2, P6 CONN_2, P7 CONN_2, P8 CONN_2, P9 CONN_2, U1 ZXRE060, U10 OPA227, U11 OP07, U12 LT1995, U13 ADG44X, U2 TEENSY3.1, U3 MAX6176AASA+, U4 LT1995, U5 AD8250, U6 MEA1D05XXSC, U7 OPA129, U8 OPA129, U9 ADG44X

Commit message: Modified schematic.  Changed +/-15V DC-DC converter to +/-12V DC-DC converter.  Changed net labels accordingly. Remade netlist, etc.
Connections:
- net +15V renamed +12V
- net -15V renamed -12V
Other:
- note added: "+/- 12V Supply for OPAMPs"
- note added: "+/- 12V supply test points"
- note removed: "+/- 15V Supply for OPAMPs"
- note removed: "+/- 15V supply test points"
Changed lines of the file:
@@
 Sheet 1 1
 Title ""
-Date "7 jan 2017"
+Date "19 dec 2018"
 Rev ""
 Comp ""
@@
 DAC_GAIN_A1
 Text Label 2975 7850 2    60   ~ 0
--15V
+-12V
 Text Label 4375 7850 0    60   ~ 0
-+15V
++12V
 Text Label 4250 1150 0    60   ~ 0
 GND
 Text Label 4375 8050 0    60   ~ 0
--15V
+-12V
 Text Label 4375 7950 0    60   ~ 0
 DAC_BIP_NX
@@
 AGND
 Text Label 900  6300 3    60   ~ 0
--15V
+-12V
 Text Label 1625 6300 3    60   ~ 0
 AGND
 Text Label 1625 5300 1    60   ~ 0
-+15V
++12V
 Text Notes 550  6950 0    60   ~ 0
 Scale bipolar DAC (DAC_BIP) by gain N=1,2,5, or 10 to get DAC_BIP_NX. Gain is selected using
@@
 $EndComp
 Text Label 2650 5800 2    60   ~ 0
--15V
+-12V
 Text Label 4350 5800 0    60   ~ 0
-+15V
++12V
 Text Label 2650 5900 2    60   ~ 0
 AGND
@@
 AGND
 Text Label 11575 8425 3    60   ~ 0
--15V
+-12V
 Text Label 12300 8425 3    60   ~ 0
 AGND
 Text Label 12300 7425 1    60   ~ 0
-+15V
++12V
 Text Notes 550  4950 0    60   ~ 0
 Amplifier Gain=1.67
@@
 GND
 Text Label 8200 15025 0    60   ~ 0
--15V
+-12V
 Text Label 8200 15225 0    60   ~ 0
-+15V
++12V
 Text Label 1800 3650 2    60   ~ 0
 5V
@@
 5V
 Text Notes 7000 14150 0    60   ~ 0
-+/- 15V Supply for OPAMPs
++/- 12V Supply for OPAMPs
 $Comp
 L OPA129 U8
@@
 	9950 8100 10250 8100
 Text Label 10250 7900 0    60   ~ 0
-+15V
++12V
 Text Label 10250 8100 0    60   ~ 0
--15V
+-12V
 Text Notes 6500 6950 0    60   ~ 0
 Uniy Gain Buffer for Reference Electrode
@@
 AGND
 Text Label 925  8525 3    60   ~ 0
--15V
+-12V
 Text Label 1650 8525 3    60   ~ 0
 AGND
 Text Label 1650 7525 1    60   ~ 0
-+15V
++12V
 Wire Wire Line
 	1075 8325 1075 8225
@@
 	9900 10500 9700 10500
 Text Label 9700 10500 2    60   ~ 0
--15V
+-12V
 Wire Wire Line
 	10800 10300 11000 10300
 Text Label 11000 10300 0    60   ~ 0
-+15V
++12V
 Text Label 11000 10400 0    60   ~ 0
 CTR_ELECT
@@
 AGND
 Text Label 12225 10825 3    60   ~ 0
--15V
+-12V
 Text Label 12950 10825 3    60   ~ 0
 AGND
 Text Label 12950 9825 1    60   ~ 0
-+15V
++12V
 Wire Wire Line
 	12375 10625 12375 10525
@@
 WRK_ELECT
 Text Label 11050 4450 0    60   ~ 0
--15V
+-12V
 Text Label 11050 4350 0    60   ~ 0
-+15V
++12V
 Text Label 11050 4550 0    60   ~ 0
 AGND
@@
 	8450 4300 8650 4300
 Text Label 8650 4100 0    60   ~ 0
-+15V
++12V
 Text Label 8650 4300 0    60   ~ 0
--15V
+-12V
 Wire Wire Line
 	7350 1550 7350 4100
@@
 	11450 1550 9650 1550
 Text Label 13600 4450 0    60   ~ 0
--15V
+-12V
 Text Label 13600 4350 0    60   ~ 0
-+15V
++12V
 Text Label 13600 4550 0    60   ~ 0
 AGND
@@
 $EndComp
 Text Label 12250 2950 2    60   ~ 0
--15V
+-12V
 Text Label 13650 2950 0    60   ~ 0
-+15V
++12V
 Text Label 12250 2650 2    60   ~ 0
 REF_0V6
@@
 AGND
 Text Label 12550 1900 3    60   ~ 0
--15V
+-12V
 Text Label 13275 1900 3    60   ~ 0
 AGND
 Text Label 13275 900  1    60   ~ 0
-+15V
++12V
 Wire Wire Line
 	12700 1700 12700 1600
@@
 AGND
 Text Label 7625 6325 3    60   ~ 0
--15V
+-12V
 Text Label 8350 6325 3    60   ~ 0
 AGND
 Text Label 8350 5325 1    60   ~ 0
-+15V
++12V
 Wire Wire Line
 	7775 6125 7775 6025
@@
 AGND
 Text Label 10150 6200 3    60   ~ 0
--15V
+-12V
 Text Label 10500 5350 1    60   ~ 0
-+15V
++12V
 Text Label 10500 6200 3    60   ~ 0
 AGND
@@
 AGND
 Text Label 12750 6250 3    60   ~ 0
--15V
+-12V
 Text Label 13100 5400 1    60   ~ 0
-+15V
++12V
 Text Label 13100 6250 3    60   ~ 0
 AGND
@@
 Connection ~ 9050 14850
 Text Label 8800 14850 2    60   ~ 0
--15V
+-12V
 $Comp
 L CONN_2 P12
@@
 Connection ~ 9050 15600
 Text Label 8800 15600 2    60   ~ 0
-+15V
++12V
 Text Notes 8100 15850 0    60   ~ 0
-+/- 15V supply test points
++/- 12V supply test points
 $Comp
 L CONN_2 P19
@@
 10V Reference voltage.
 Text Label 2750 12550 2    60   ~ 0
-+15V
++12V
 Text Label 2750 12750 2    60   ~ 0
 GND
@@
 	7450 12450 7450 12200
 Text Label 7050 12200 1    60   ~ 0
-+15V
++12V
 Text Label 7450 12200 1    60   ~ 0
--15V
+-12V
 $Comp
 L R R4
@@
 	11650 12750 11900 12750
 Text Label 11900 12750 0    60   ~ 0
-+15V
++12V
 Text Label 10400 12950 2    60   ~ 0
--15V
+-12V
 Wire Wire Line
 	10050 12650 10050 13050
@@
 GND
 Text Label 1900 12150 1    60   ~ 0
-+15V
++12V
 $Comp
 L CONN_2 P1
