File: hardware/pcbs/multiplexer_adapters/mux_to_3pin/adapter.kicad_pcb (KiCad board)
At the start: 2 copper layers, 26.7 x 50.8 mm, 8 parts, among them K1 CONN_3, K2 CONN_3, K3 CONN_3, K4 CONN_3, K5 CONN_3, K6 CONN_3, K7 CONN_3, P1 CONN_5X2

Commit message: Final checkin before order prototypes of multiplexer_v2, mux_to_3pin and mux_to_term pcbs.
Other:
- board text removed: "WRK2"
Changed lines of the file:
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@@
   (general
     (links 21)
-    (no_connects 21)
+    (no_connects 0)
     (area 32.334288 50.736499 90.855713 101.663501)
     (thickness 1.6)
@@
     )
   )
+  (dimension 26.67 (width 0.2032) (layer Dwgs.User)
+    (gr_text "1.0500 in" (at 64.135 109.372399) (layer Dwgs.User)
+      (effects (font (size 1.016 1.016) (thickness 0.2032)))
+    )
+    (feature1 (pts (xy 77.47 88.9) (xy 77.47 110.286799)))
+    (feature2 (pts (xy 50.8 88.9) (xy 50.8 110.286799)))
+    (crossbar (pts (xy 50.8 108.457999) (xy 77.47 108.457999)))
+    (arrow1a (pts (xy 77.47 108.457999) (xy 76.343497 109.044419)))
+    (arrow1b (pts (xy 77.47 108.457999) (xy 76.343497 107.871579)))
+    (arrow2a (pts (xy 50.8 108.457999) (xy 51.926503 109.044419)))
+    (arrow2b (pts (xy 50.8 108.457999) (xy 51.926503 107.871579)))
+  )
   (gr_text WK7 (at 74.93 92.202 90) (layer F.SilkS)
     (effects (font (size 1.016 1.016) (thickness 0.2032)))
@@
     (effects (font (size 1.016 1.016) (thickness 0.2032)))
   )
-  (gr_text WRK2 (at 75.184 61.468) (layer B.SilkS)
-    (effects (font (size 1.016 1.016) (thickness 0.2032)) (justify mirror))
-  )
   (gr_text REF (at 72.39 60.706 90) (layer F.SilkS)
