File: hardware/pcbs/multiplexer_adapters/mux_to_term/adapter.kicad_pcb (KiCad board)
At the start: 2 copper layers, 26.7 x 50.8 mm, 3 parts, among them K1 CONN_3, P1 CONN_5X2, P2 CONN_7

Commit message: Final checkin before order prototypes of multiplexer_v2, mux_to_3pin and mux_to_term pcbs.
Other:
- board text added: "Rodeostat Multiplexer Screw Terminal Adapter V0.1 R1 www.iorodeo.com"
- board text removed: "Rodeostat Multiplexer Screw Terminal Adapter V0.1 www.iorodeo.com"
Changed lines of the file:
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@@
     (area 32.334288 50.736499 90.855713 101.663501)
     (thickness 1.6)
-    (drawings 30)
+    (drawings 31)
     (tracks 33)
     (zones 0)
@@
     )
   )
+  (dimension 26.67 (width 0.2032) (layer Dwgs.User)
+    (gr_text "1.0500 in" (at 64.135 108.864399) (layer Dwgs.User)
+      (effects (font (size 1.016 1.016) (thickness 0.2032)))
+    )
+    (feature1 (pts (xy 77.47 88.392) (xy 77.47 109.778799)))
+    (feature2 (pts (xy 50.8 88.392) (xy 50.8 109.778799)))
+    (crossbar (pts (xy 50.8 107.949999) (xy 77.47 107.949999)))
+    (arrow1a (pts (xy 77.47 107.949999) (xy 76.343497 108.536419)))
+    (arrow1b (pts (xy 77.47 107.949999) (xy 76.343497 107.363579)))
+    (arrow2a (pts (xy 50.8 107.949999) (xy 51.926503 108.536419)))
+    (arrow2b (pts (xy 50.8 107.949999) (xy 51.926503 107.363579)))
+  )
   (gr_text WRK7 (at 65.532 95.6945) (layer F.SilkS)
     (effects (font (size 1.016 1.016) (thickness 0.2032)) (justify left))
@@
     (effects (font (size 1.016 1.016) (thickness 0.2032)) (justify left))
   )
-  (gr_text "Rodeostat Multiplexer \nScrew Terminal Adapter V0.1\nwww.iorodeo.com" (at 65.532 77.216 90) (layer B.SilkS)
+  (gr_text "Rodeostat Multiplexer \nScrew Terminal Adapter V0.1 R1\nwww.iorodeo.com" (at 65.532 77.216 90) (layer B.SilkS)
     (effects (font (size 1.016 1.016) (thickness 0.2032)) (justify mirror))
   )
