File: hardware/pcbs/itsy_bitsy_m4_shield_v0p1/potentiostat.sch (KiCad schematic (older format))
At the start: 137 parts, among them K1 Conn_01x03, P1 Conn_01x02, P10 Conn_01x02, P11 Conn_01x02, P12 Conn_01x02, P13 Conn_02x05_Odd_Even, P14 Conn_02x05_Odd_Even, P15 Conn_02x02_Odd_Even, P16 Conn_02x02_Odd_Even, P17 Conn_01x02, P18 Conn_01x02, P19 Conn_01x02, P2 Conn_01x02, P20 Conn_01x02, P21 Conn_01x02, P22 Conn_01x02, P3 Conn_01x02, P4 Conn_01x02, P5 Conn_01x02, P6 Conn_01x02, P7 Conn_01x02, P8 Conn_01x02, P9 Conn_01x02, U1 74HC138, U10 REF33XX, U11 OP07, U12 OP07, U13 OP07, U14 OP07, U15 OP07, U16 OP07, U17 OP07, U18 OP07, U19 74HC138, U2 ITSY_BITSY_M4, U20 OP07, U21 74HC138, U3 DG411xY, U4 DG411xY, U5 DG411xY, U6 MEA1D05XXSC, U7 DG411xY, U8 DG411xY, U9 TL072

Commit message: Created gerber files for itsy bitsy MX shield.
Other:
- note added: "Note: ITSY_BITSY_M0 also works."
Changed lines of the file:
@@
 NoConn ~ 2850 2700
 NoConn ~ 2950 2700
+Text Notes 3525 900  0    50   ~ 0
+Note: ITSY_BITSY_M0 also works.
 $EndSCHEMATC
