File: hardware/pcbs/itsy_bitsy_mx_shield_v0p1/potentiostat.sch (KiCad schematic (older format))
At the start: 137 parts, among them K1 Conn_01x03, P1 Conn_01x02, P10 Conn_01x02, P11 Conn_01x02, P12 Conn_01x02, P13 Conn_02x05_Odd_Even, P14 Conn_02x05_Odd_Even, P15 Conn_02x02_Odd_Even, P16 Conn_02x02_Odd_Even, P17 Conn_01x02, P18 Conn_01x02, P19 Conn_01x02, P2 Conn_01x02, P20 Conn_01x02, P21 Conn_01x02, P22 Conn_01x02, P3 Conn_01x02, P4 Conn_01x02, P5 Conn_01x02, P6 Conn_01x02, P7 Conn_01x02, P8 Conn_01x02, P9 Conn_01x02, U1 74HC138, U10 REF33XX, U11 OP07, U12 OP07, U13 OP07, U14 OP07, U15 OP07, U16 OP07, U17 OP07, U18 OP07, U19 74HC138, U2 ITSY_BITSY_M4, U20 OP07, U21 74HC138, U3 DG411xY, U4 DG411xY, U5 DG411xY, U6 MEA1D05XXSC, U7 DG411xY, U8 DG411xY, U9 TL072

Commit message: Re-routed board and remade gerber files.
Connections:
- net labels added: A3_D17, D7
- net labels removed: A1_D15, A4_D18, A5_D19
- wire segments 639 -> 643
- no-connect marks 45 -> 41
Changed lines of the file:
@@
 	19325 16725 19525 16725
 Wire Wire Line
-	19525 16825 19325 16825
-Wire Wire Line
 	20025 16625 20225 16625
 Wire Wire Line
@@
 Text Label 3750 2150 0    60   ~ 0
 SDA
-Text Label 3750 2050 0    60   ~ 0
-SCL
 Wire Wire Line
-	2350 1750 2150 1750
+	2350 1650 2150 1650
 Text Label 3750 1750 0    60   ~ 0
 TIA_GAIN_A0
@@
 TIA_GAIN_A1
 Wire Wire Line
-	3550 1950 3750 1950
+	2350 1850 2150 1850
 Wire Wire Line
-	3550 1850 3750 1850
-Text Label 3750 1950 0    50   ~ 0
+	2350 1950 2150 1950
+Text Label 2150 1850 2    60   ~ 0
 REF_GAIN_A0
-Text Label 3750 1850 0    50   ~ 0
+Text Label 2150 1950 2    60   ~ 0
 REF_GAIN_A1
 Wire Wire Line
@@
 NoConn ~ 2350 1250
 NoConn ~ 2350 1350
-Text Label 2150 1750 2    60   ~ 0
+Text Label 2150 1650 2    60   ~ 0
 REF_ELECT_UNI
 Wire Wire Line
-	2150 1650 2350 1650
+	2150 1550 2350 1550
 Text Label 2150 2050 2    60   ~ 0
 SCK
 Wire Wire Line
 	2350 2050 2150 2050
-Text Label 2150 1650 2    60   ~ 0
+Text Label 2150 1550 2    60   ~ 0
 TIA_OUT_UNI
 NoConn ~ 3550 1050
@@
 Wire Wire Line
 	3550 2350 3750 2350
-Text Label 3750 2250 0    50   ~ 0
+Text Label 3750 2250 0    60   ~ 0
 TX_D1
-Text Label 3750 2350 0    50   ~ 0
+Text Label 3750 2350 0    60   ~ 0
 RX_D0
-Text Label 2150 1950 2    50   ~ 0
-A5_D19
-Wire Wire Line
-	2350 1950 2150 1950
 Wire Wire Line
-	2350 1850 2150 1850
-Wire Wire Line
-	2350 1550 2125 1550
-Text Label 2150 1850 2    50   ~ 0
-A4_D18
-Text Label 2125 1550 2    50   ~ 0
-A1_D15
+	2350 1750 2125 1750
+Text Label 2125 1750 2    60   ~ 0
+A3_D17
 Text Label 19325 16725 2    50   ~ 0
-A1_D15
+D7
 Text Label 20225 16725 0    50   ~ 0
-A4_D18
-Text Label 19325 16825 2    50   ~ 0
-A5_D19
-NoConn ~ 20025 16825
-NoConn ~ 20025 16925
-NoConn ~ 20025 17025
-NoConn ~ 19525 17025
-NoConn ~ 19525 16925
+A3_D17
 NoConn ~ 2750 2700
 NoConn ~ 2850 2700
@@
 Text Notes 3525 900  0    50   ~ 0
 Note: ITSY_BITSY_M0 also works.
+Text Label 3750 1850 0    60   ~ 0
+D7
+Text Label 3750 2050 0    60   ~ 0
+SCL
+Wire Wire Line
+	3550 1850 3750 1850
+NoConn ~ 3550 1950
+Text Label 19325 17025 2    60   ~ 0
+SCK
+Text Label 19325 16925 2    60   ~ 0
+POCI
+Text Label 19325 16825 2    60   ~ 0
+SCL
+Wire Wire Line
+	19525 17025 19325 17025
+Wire Wire Line
+	19525 16925 19325 16925
+Wire Wire Line
+	19525 16825 19325 16825
+Text Label 20225 17025 0    60   ~ 0
+CS
+Text Label 20225 16925 0    60   ~ 0
+PICO
+Text Label 20225 16825 0    60   ~ 0
+SDA
+Wire Wire Line
+	20025 17025 20225 17025
+Wire Wire Line
+	20025 16925 20225 16925
+Wire Wire Line
+	20025 16825 20225 16825
 $EndSCHEMATC

Commit message: Fixed footprint issue with mx design.
Parts:
- P1, P2, P3: footprint pin_array:PIN_ARRAY_2X1 -> ost_connblocks:CONNBLOCK2
Changed lines of the file:
@@
 F 0 "P1" H 8530 13442 50  0000 L CNN
 F 1 "Conn_01x02" H 8530 13351 50  0000 L CNN
-F 2 "pin_array:PIN_ARRAY_2X1" H 8450 13450 50  0001 C CNN
+F 2 "ost_connblocks:CONNBLOCK2" H 8450 13450 50  0001 C CNN
 F 3 "~" H 8450 13450 50  0001 C CNN
 	1    8450 13450
@@
 F 0 "P2" H 8530 14392 50  0000 L CNN
 F 1 "Conn_01x02" H 8530 14301 50  0000 L CNN
-F 2 "pin_array:PIN_ARRAY_2X1" H 8450 14400 50  0001 C CNN
+F 2 "ost_connblocks:CONNBLOCK2" H 8450 14400 50  0001 C CNN
 F 3 "~" H 8450 14400 50  0001 C CNN
 	1    8450 14400
@@
 F 0 "P3" H 8530 15392 50  0000 L CNN
 F 1 "Conn_01x02" H 8530 15301 50  0000 L CNN
-F 2 "pin_array:PIN_ARRAY_2X1" H 8450 15400 50  0001 C CNN
+F 2 "ost_connblocks:CONNBLOCK2" H 8450 15400 50  0001 C CNN
 F 3 "~" H 8450 15400 50  0001 C CNN
 	1    8450 15400

Commit message: Modified amplifier gains for mx design to support 3.3V analog ranges.
Parts:
- removed C1: 4.7uF, Capacitor_SMD:C_0603_1608Metric, symbol Device:C
- removed U10: REF33XX, Package_TO_SOT_SMD:SOT-23, symbol REF33XX:REF33XX
- R1, R2, R26, R28: value 12k -> 33k
- R14: value 300k -> 250k
- R15: value 30k -> 25k
- R16: value 3k -> 2.5k
- R17: value 300 -> 250
- R27: value 10k -> 5k
- R29: value 20k -> 33k
- R33, R34, R36: value 12k -> 10k
- R4: value 100k -> 20k
- R6: value 20k -> 10k
Connections:
- net labels added: REF_1V65, REF_NEG_1V65
- net labels removed: REF_0V6, REF_3V, REF_NEG_0V6
- wire segments 643 -> 636
Other:
- note added: "1. Replace w/ 20k\nDONE"
- note added: "1.65V reference test points"
- note added: "2. Replace w/ 10k\nDONE"
- note added: "3. Remove U10 and C1. \nOnly need 3.3V reference now. \nDONE"
- note added: "4. Replace References REF_1V65 and REF_NEG_0V6 with\nREF_1V65 and REF_NEG_1V65\nDONE"
- note added: "5. Change R5 and R3 to 20k\nChange R1 and R2 to 33k\nDone"
- note added: "6. Change gain resistors \nR14, R15, R16, R17 to \n250k, 25k, 2.5k and 250\nDONE"
- note added: "7. Replace R27 with 5K and R29 with 33k\nDONE"
- note added: "8. Replace R26 and R28 with 33k\nDONE"
- note added: "9. Replace R33, R34, R36 with 10k resistors\nDONE"
- note added: "Change Notes:\n------------------------\n\n1. (Done) Change R4 from 100k to 20k\n2. (Done) Change R6 from 20k to 10k \n3. (Done) Remove Reference voltage U10 and C1. Only need 3.3V reference now. \n4. (Done) Change all instances of REF_1V65 to REF_1V65\n5. (Done) Change R5 and R3 to 20k and also Change R1 and R2 to 33k\n6. (Done) Change gain resistors R14, R15, R16, R17 to 250k, 25k, 2.5k and 250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"
- note added: "Scale 3.3V to create -1.65V reference"
- note added: "Shift and scale unipolar DAC (DAC_UNI) from [0V, 3.3V] \nrange to bipolar DAC (DAC_BIP) in [-1V, 1V] range. \n"
- note added: "invert to create +1.65V reference"
- note added: "scale TIA signal by 6.6x"
- note added: "shift TIA signal to 0-3.3V range"
- note added: "transimpedance amplifier with selectable gain using kelvin switching\nsee http://www.analog.com/library/analogdialogue/archives/47-05/pgtia.html\n\nSet gains so that output voltage range is -0.25V to 0.25V. \nInput current ranges (+/-) 1uA, 10uA, 100uA, 1000uA \n"
- note removed: "0.6V reference test points"
- note removed: "Shift and scales unipolar DAC (DAC_UNI) from [0V,1.2V] \nrange to bipolar DAC (DAC_BIP) in [-1V,1V] range. \n"
- note removed: "inverts -0.6V reference to \ncreate 0.6V reference"
- note removed: "scale TIA signal by 2x"
- note removed: "scales 3V reference to \ncreate -0.6V reference"
- note removed: "shift TIA signal to 0-1.2V range"
- note removed: "transimpedance amplifier with selectable gain using kelvin switching\nsee http://www.analog.com/library/analogdialogue/archives/47-05/pgtia.html\n\nSet gains so that output voltage range is -0.6V to 0.6V. \nInput current ranges (+/-) 1uA, 10uA, 100uA, 1000uA \n"
- moved on the sheet: C12, C15, C18, C21, C5, R13, R4, R6, R8, U12, U14

Commit message: Worked on layout, re-routing and BOM.
Parts:
- C25, C26, C27, C28: value 68nF -> 56nF
Other:
- note added: "4. Replace References REF_0V6 and REF_NEG_0V6 with\nREF_1V65 and REF_NEG_1V65\nDONE"
- note removed: "4. Replace References REF_1V65 and REF_NEG_0V6 with\nREF_1V65 and REF_NEG_1V65\nDONE"
Changed lines of the file:
@@
 P 13175 1350
 F 0 "C25" V 13075 1200 50  0000 C CNN
-F 1 "68nF" V 13075 1500 50  0000 C CNN
+F 1 "56nF" V 13075 1500 50  0000 C CNN
 F 2 "Capacitor_SMD:C_0603_1608Metric" H 13213 1200 50  0001 C CNN
 F 3 "~" H 13175 1350 50  0001 C CNN
@@
 P 13225 4700
 F 0 "C28" V 13125 4550 50  0000 C CNN
-F 1 "68nF" V 13125 4850 50  0000 C CNN
+F 1 "56nF" V 13125 4850 50  0000 C CNN
 F 2 "Capacitor_SMD:C_0603_1608Metric" H 13263 4550 50  0001 C CNN
 F 3 "~" H 13225 4700 50  0001 C CNN
@@
 P 13175 2500
 F 0 "C26" V 13075 2350 50  0000 C CNN
-F 1 "68nF" V 13075 2650 50  0000 C CNN
+F 1 "56nF" V 13075 2650 50  0000 C CNN
 F 2 "Capacitor_SMD:C_0603_1608Metric" H 13213 2350 50  0001 C CNN
 F 3 "~" H 13175 2500 50  0001 C CNN
@@
 P 13175 3650
 F 0 "C27" V 13075 3500 50  0000 C CNN
-F 1 "68nF" V 13075 3800 50  0000 C CNN
+F 1 "56nF" V 13075 3800 50  0000 C CNN
 F 2 "Capacitor_SMD:C_0603_1608Metric" H 13213 3500 50  0001 C CNN
 F 3 "~" H 13175 3650 50  0001 C CNN
@@
 $EndComp
 Text Notes 3250 9925 0    50   ~ 10
-4. Replace References REF_1V65 and REF_NEG_0V6 with\nREF_1V65 and REF_NEG_1V65\nDONE
+4. Replace References REF_0V6 and REF_NEG_0V6 with\nREF_1V65 and REF_NEG_1V65\nDONE
 Text Notes 11275 2950 0    50   ~ 10
 6. Change gain resistors \nR14, R15, R16, R17 to \n250k, 25k, 2.5k and 250\nDONE

Commit message: Added gerber files for rodeostat mx V0.1 R3. Added fab files.
Parts:
- R14: value 250k -> 300k
- R15: value 25k -> 30k
- R16: value 2.5k -> 3k
- R17: value 250 -> 300
- R27: value 5k -> 2k
- R29: value 33k -> 11k
Other:
- note added: "6. Replace R27 with 2k and R29 with 11k\nDONE\n"
- note added: "7. Replace R26 and R28 with 33k\nDONE"
- note added: "8. Replace R33, R34, R36 with 10k resistors\nDONE"
- note added: "Change Notes:\n------------------------\n\n1. (Done) Change R4 from 100k to 20k\n2. (Done) Change R6 from 20k to 10k \n3. (Done) Remove Reference voltage U10 and C1. Only need 3.3V reference now. \n4. (Done) Change all instances of REF_1V65 to REF_1V65\n5. (Done) Change R5 and R3 to 20k and also Change R1 and R2 to 33k\n6. (Done) Replace R27 with 5K and R29 with 33k\n7. (Done) Replace R26 and R28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"
- note added: "scale TIA signal by 5.5x"
- note added: "transimpedance amplifier with selectable gain using kelvin switching\nsee http://www.analog.com/library/analogdialogue/archives/47-05/pgtia.html\n\nSet gains so that output voltage range is -0.3V to 0.3V. \nInput current ranges (+/-) 1uA, 10uA, 100uA, 1000uA \n"
- note removed: "6. Change gain resistors \nR14, R15, R16, R17 to \n250k, 25k, 2.5k and 250\nDONE"
- note removed: "7. Replace R27 with 5K and R29 with 33k\nDONE"
- note removed: "8. Replace R26 and R28 with 33k\nDONE"
- note removed: "9. Replace R33, R34, R36 with 10k resistors\nDONE"
- note removed: "Change Notes:\n------------------------\n\n1. (Done) Change R4 from 100k to 20k\n2. (Done) Change R6 from 20k to 10k \n3. (Done) Remove Reference voltage U10 and C1. Only need 3.3V reference now. \n4. (Done) Change all instances of REF_1V65 to REF_1V65\n5. (Done) Change R5 and R3 to 20k and also Change R1 and R2 to 33k\n6. (Done) Change gain resistors R14, R15, R16, R17 to 250k, 25k, 2.5k and 250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"
- note removed: "scale TIA signal by 6.6x"
- note removed: "transimpedance amplifier with selectable gain using kelvin switching\nsee http://www.analog.com/library/analogdialogue/archives/47-05/pgtia.html\n\nSet gains so that output voltage range is -0.25V to 0.25V. \nInput current ranges (+/-) 1uA, 10uA, 100uA, 1000uA \n"
Changed lines of the file:
@@
 P 13175 1650
 F 0 "R14" V 13275 1625 50  0000 C CNN
-F 1 "250k" V 13175 1650 50  0000 C CNN
+F 1 "300k" V 13175 1650 50  0000 C CNN
 F 2 "Resistor_SMD:R_0603_1608Metric" V 13105 1650 50  0001 C CNN
 F 3 "~" H 13175 1650 50  0001 C CNN
@@
 P 13225 5000
 F 0 "R17" V 13325 4975 50  0000 C CNN
-F 1 "250" V 13225 4975 50  0000 C CNN
+F 1 "300" V 13225 4975 50  0000 C CNN
 F 2 "Resistor_SMD:R_0603_1608Metric" V 13155 5000 50  0001 C CNN
 F 3 "~" H 13225 5000 50  0001 C CNN
@@
 P 13175 2800
 F 0 "R15" V 13275 2775 50  0000 C CNN
-F 1 "25k" V 13175 2775 50  0000 C CNN
+F 1 "30k" V 13175 2775 50  0000 C CNN
 F 2 "Resistor_SMD:R_0603_1608Metric" V 13105 2800 50  0001 C CNN
 F 3 "~" H 13175 2800 50  0001 C CNN
@@
 P 13175 3950
 F 0 "R16" V 13275 3925 50  0000 C CNN
-F 1 "2.5k" V 13175 3925 50  0000 C CNN
+F 1 "3k" V 13175 3925 50  0000 C CNN
 F 2 "Resistor_SMD:R_0603_1608Metric" V 13105 3950 50  0001 C CNN
 F 3 "~" H 13175 3950 50  0001 C CNN
@@
 P 18175 5500
 F 0 "R27" V 18075 5500 50  0000 C CNN
-F 1 "5k" V 18175 5500 50  0000 C CNN
+F 1 "2k" V 18175 5500 50  0000 C CNN
 F 2 "Resistor_SMD:R_0603_1608Metric" V 18105 5500 50  0001 C CNN
 F 3 "~" H 18175 5500 50  0001 C CNN
@@
 P 19150 4850
 F 0 "R29" V 19050 4850 50  0000 C CNN
-F 1 "33k" V 19150 4850 50  0000 C CNN
+F 1 "11k" V 19150 4850 50  0000 C CNN
 F 2 "Resistor_SMD:R_0603_1608Metric" V 19080 4850 50  0001 C CNN
 F 3 "~" H 19150 4850 50  0001 C CNN
@@
 scale buffered reference electrode voltage\n according to gain setting
 Text Notes 18900 6350 0    60   ~ 0
-scale TIA signal by 6.6x
+scale TIA signal by 5.5x
 Text Notes 21925 6350 0    60   ~ 0
 shift TIA signal to 0-3.3V range
@@
 Scale bipolar DAC (DAC_BIP) by gain N=1,2,5, or 10  to get DAC_BIP_NX. \nGain is selected using DAC_GAIN_A0 and DAC_GAIN_A1
 Text Notes 13650 6525 0    60   ~ 0
-transimpedance amplifier with selectable gain using kelvin switching\nsee http://www.analog.com/library/analogdialogue/archives/47-05/pgtia.html\n\nSet gains so that output voltage range is -0.25V to 0.25V. \nInput current ranges (+/-)  1uA, 10uA, 100uA, 1000uA \n
+transimpedance amplifier with selectable gain using kelvin switching\nsee http://www.analog.com/library/analogdialogue/archives/47-05/pgtia.html\n\nSet gains so that output voltage range is -0.3V to 0.3V. \nInput current ranges (+/-)  1uA, 10uA, 100uA, 1000uA \n
 $Comp
 L Analog_Switch:DG411xY U4
@@
 5. Change R5 and R3 to 20k\nChange R1 and R2 to 33k\nDone
 Text Notes 17975 4750 0    50   ~ 10
-7. Replace R27 with 5K and R29 with 33k\nDONE
+6. Replace R27 with 2k and R29 with 11k\nDONE\n
 Text Notes 17125 12175 0    50   ~ 10
-8. Replace R26 and R28 with 33k\nDONE
+7. Replace R26 and R28 with 33k\nDONE
 Text Notes 675  -125 0    250  ~ 0
-Change Notes:\n------------------------\n\n1. (Done) Change R4 from 100k to 20k\n2. (Done) Change R6 from 20k to 10k \n3. (Done) Remove Reference voltage U10 and C1.  Only need 3.3V reference now. \n4. (Done) Change all instances of REF_1V65 to REF_1V65\n5. (Done) Change R5 and R3 to 20k and also Change R1 and R2 to 33k\n6. (Done) Change gain resistors  R14, R15, R16, R17 to 250k, 25k, 2.5k and 250\n7. (Done) Replace R27 with 5K and R29 with 33k\n8. (Done) Replace R26 and R28 with 33k\n9. (Done) Replace R33, R34, R36  with 10k resistors\n\n-----------------------------------------------------------------------------\nExplaination\nItems 1,2 and 3 change reference voltages to +/- 1.65V\nItem 5 modifies amplifier so [0V, 3.3V]  is scaled and shifted to [-1V, 1V]\nItem 6 Changes gains of transimpedance amplifiers so that all current ranges maps to  goes to [-0.25V, 0.25V]\nItem 7 Changes gain of post transimpedace amplifier stage to 6.6 so that is scale [-0.25V, 0.25V] to [-1.65V, 1.65V]\nItem 8 modifies summing amplifier so that it maps [-1V, 1V] to [-1.65V, 1.65V]\nItem 9 doesn't change anything .. just reduces number of resistor types used. \n\n\n
+Change Notes:\n------------------------\n\n1. (Done) Change R4 from 100k to 20k\n2. (Done) Change R6 from 20k to 10k \n3. (Done) Remove Reference voltage U10 and C1.  Only need 3.3V reference now. \n4. (Done) Change all instances of REF_1V65 to REF_1V65\n5. (Done) Change R5 and R3 to 20k and also Change R1 and R2 to 33k\n6. (Done) Replace R27 with 5K and R29 with 33k\n7. (Done) Replace R26 and R28 with 33k\n8. (Done) Replace R33, R34, R36  with 10k resistors\n\n-----------------------------------------------------------------------------\nExplaination\nItems 1,2 and 3 change reference voltages to +/- 1.65V\nItem 5 modifies amplifier so [0V, 3.3V]  is scaled and shifted to [-1V, 1V]\nItem 6 Changes gain of post transimpedace amplifier stage to 6.6 so that is scale [-0.25V, 0.25V] to [-1.65V, 1.65V]\nItem 7 modifies summing amplifier so that it maps [-1V, 1V] to [-1.65V, 1.65V]\nItem 8 doesn't change anything .. just reduces number of resistor types used. \n\n\n
 Text Notes 600  10400 0    50   ~ 10
 3. Remove U10 and C1.  \nOnly need 3.3V reference now. \nDONE
@@
 Text Notes 3250 9925 0    50   ~ 10
 4. Replace References REF_0V6 and REF_NEG_0V6 with\nREF_1V65 and REF_NEG_1V65\nDONE
-Text Notes 11275 2950 0    50   ~ 10
-6. Change gain resistors \nR14, R15, R16, R17 to \n250k, 25k, 2.5k and 250\nDONE
 Text Notes 2050 10025 0    50   ~ 10
 2. Replace w/ 10k\nDONE
 Text Notes 21300 4325 0    50   ~ 10
-9. Replace R33, R34, R36  with 10k resistors\nDONE
+8. Replace R33, R34, R36  with 10k resistors\nDONE
 $EndSCHEMATC
