File: hardware/pcbs/itsy_bitsy_mx_shield_v0p1/high_current/potentiostat.sch (KiCad schematic (older format))
At the start: 135 parts, among them K1 Conn_01x03, P1 Conn_01x02, P10 Conn_01x02, P11 Conn_01x02, P12 Conn_01x02, P13 Conn_02x05_Odd_Even, P14 Conn_02x05_Odd_Even, P15 Conn_02x02_Odd_Even, P16 Conn_02x02_Odd_Even, P17 Conn_01x02, P18 Conn_01x02, P19 Conn_01x02, P2 Conn_01x02, P20 Conn_01x02, P21 Conn_01x02, P22 Conn_01x02, P3 Conn_01x02, P4 Conn_01x02, P5 Conn_01x02, P6 Conn_01x02, P7 Conn_01x02, P8 Conn_01x02, P9 Conn_01x02, U1 74HC138, U11 OP07, U12 OP07, U13 OP07, U14 OP07, U15 OP07, U16 OP07, U17 OP07, U18 OP07, U19 74HC138, U2 ITSY_BITSY_M4, U20 OP07, U21 74HC138, U3 DG411xY, U4 DG411xY, U5 DG411xY, U6 MEA1D05XXSC, U7 DG411xY, U8 DG411xY, U9 TL072

Commit message: Added fab files to include through hole assembly.
Increased revision number V0.1 R4.  Remade gerbers to include addtional
elements on silkscreen.
Parts:
- added UA2, UB2: header_14_pos, dummy:header_14_pos, symbol dummy:header_14_pos
- added UC2: header_5_pos, dummy:header_5_pos, symbol dummy:header_5_pos
Other:
- note added: "Dummy headers \nfor auto assembly"
- moved on the sheet: C7, C8, C9
Changed lines of the file:
@@
 Text Notes 7675 16950 0    60   ~ 0
 electrode connections
-Text Label 7125 2825 2    60   ~ 0
+Text Label 6250 2775 2    60   ~ 0
 GND
-Text Label 7125 3125 2    60   ~ 0
+Text Label 6250 3075 2    60   ~ 0
 GND
 Text Label 9375 11400 2    60   ~ 0
 REF_1V65
-Text Notes 7125 3425 0    60   ~ 0
+Text Notes 6250 3375 0    60   ~ 0
 GND test points
 Text Notes 8750 9275 0    60   ~ 0
@@
 L Device:C C9
 U 1 1 61C14C4B
-P 8050 1400
-F 0 "C9" H 8165 1446 50  0000 L CNN
-F 1 "2.2uF" H 8165 1355 50  0000 L CNN
-F 2 "Capacitor_SMD:C_0603_1608Metric" H 8088 1250 50  0001 C CNN
-F 3 "~" H 8050 1400 50  0001 C CNN
-	1    8050 1400
+P 7175 1350
+F 0 "C9" H 7290 1396 50  0000 L CNN
+F 1 "2.2uF" H 7290 1305 50  0000 L CNN
+F 2 "Capacitor_SMD:C_0603_1608Metric" H 7213 1200 50  0001 C CNN
+F 3 "~" H 7175 1350 50  0001 C CNN
+	1    7175 1350
 	1    0    0    -1
 $EndComp
-Text Label 8050 1100 1    60   ~ 0
+Text Label 7175 1050 1    60   ~ 0
 3V3
 Wire Wire Line
-	8050 1550 8050 1750
-Text Label 8050 1750 3    60   ~ 0
+	7175 1500 7175 1700
+Text Label 7175 1700 3    60   ~ 0
 GND
 Wire Wire Line
-	8050 1100 8050 1250
+	7175 1050 7175 1200
 $Comp
 L Device:C C8
 U 1 1 61D1D9C4
-P 7500 1400
-F 0 "C8" H 7615 1446 50  0000 L CNN
-F 1 "2.2uF" H 7615 1355 50  0000 L CNN
-F 2 "Capacitor_SMD:C_0603_1608Metric" H 7538 1250 50  0001 C CNN
-F 3 "~" H 7500 1400 50  0001 C CNN
-	1    7500 1400
+P 6625 1350
+F 0 "C8" H 6740 1396 50  0000 L CNN
+F 1 "2.2uF" H 6740 1305 50  0000 L CNN
+F 2 "Capacitor_SMD:C_0603_1608Metric" H 6663 1200 50  0001 C CNN
+F 3 "~" H 6625 1350 50  0001 C CNN
+	1    6625 1350
 	1    0    0    -1
 $EndComp
-Text Label 7500 1100 1    60   ~ 0
+Text Label 6625 1050 1    60   ~ 0
 3V3
 Wire Wire Line
-	7500 1550 7500 1750
-Text Label 7500 1750 3    60   ~ 0
+	6625 1500 6625 1700
+Text Label 6625 1700 3    60   ~ 0
 GND
 Wire Wire Line
-	7500 1100 7500 1250
+	6625 1050 6625 1200
 $Comp
 L Device:C C22
@@
 L Connector_Generic:Conn_01x02 P4
 U 1 1 65A7D907
-P 7675 2775
-F 0 "P4" H 7755 2767 50  0000 L CNN
-F 1 "Conn_01x02" H 7755 2676 50  0000 L CNN
-F 2 "pin_array:PIN_ARRAY_2X1" H 7675 2775 50  0001 C CNN
-F 3 "~" H 7675 2775 50  0001 C CNN
-	1    7675 2775
+P 6800 2725
+F 0 "P4" H 6880 2717 50  0000 L CNN
+F 1 "Conn_01x02" H 6880 2626 50  0000 L CNN
+F 2 "pin_array:PIN_ARRAY_2X1" H 6800 2725 50  0001 C CNN
+F 3 "~" H 6800 2725 50  0001 C CNN
+	1    6800 2725
 	1    0    0    -1
 $EndComp
@@
 L Connector_Generic:Conn_01x02 P5
 U 1 1 65A7EAED
-P 7675 3075
-F 0 "P5" H 7755 3067 50  0000 L CNN
-F 1 "Conn_01x02" H 7755 2976 50  0000 L CNN
-F 2 "pin_array:PIN_ARRAY_2X1" H 7675 3075 50  0001 C CNN
-F 3 "~" H 7675 3075 50  0001 C CNN
-	1    7675 3075
+P 6800 3025
+F 0 "P5" H 6880 3017 50  0000 L CNN
+F 1 "Conn_01x02" H 6880 2926 50  0000 L CNN
+F 2 "pin_array:PIN_ARRAY_2X1" H 6800 3025 50  0001 C CNN
+F 3 "~" H 6800 3025 50  0001 C CNN
+	1    6800 3025
 	1    0    0    -1
 $EndComp
 Wire Wire Line
-	7475 2775 7375 2775
+	6600 2725 6500 2725
 Wire Wire Line
-	7375 2775 7375 2825
+	6500 2725 6500 2775
 Wire Wire Line
-	7375 2875 7475 2875
+	6500 2825 6600 2825
 Wire Wire Line
-	7475 3075 7375 3075
+	6600 3025 6500 3025
 Wire Wire Line
-	7375 3075 7375 3125
+	6500 3025 6500 3075
 Wire Wire Line
-	7375 3175 7475 3175
+	6500 3125 6600 3125
 Wire Wire Line
-	7375 2825 7125 2825
-Connection ~ 7375 2825
+	6500 2775 6250 2775
+Connection ~ 6500 2775
 Wire Wire Line
-	7375 2825 7375 2875
+	6500 2775 6500 2825
 Wire Wire Line
-	7375 3125 7125 3125
-Connection ~ 7375 3125
+	6500 3075 6250 3075
+Connection ~ 6500 3075
 Wire Wire Line
-	7375 3125 7375 3175
+	6500 3075 6500 3125
 Text Label 2150 1450 2    60   ~ 0
 DAC_UNI
@@
 L Device:C C7
 U 1 1 668AE80C
-P 6950 1400
-F 0 "C7" H 7065 1446 50  0000 L CNN
-F 1 "2.2uF" H 7065 1355 50  0000 L CNN
-F 2 "Capacitor_SMD:C_0603_1608Metric" H 6988 1250 50  0001 C CNN
-F 3 "~" H 6950 1400 50  0001 C CNN
-	1    6950 1400
+P 6075 1350
+F 0 "C7" H 6190 1396 50  0000 L CNN
+F 1 "2.2uF" H 6190 1305 50  0000 L CNN
+F 2 "Capacitor_SMD:C_0603_1608Metric" H 6113 1200 50  0001 C CNN
+F 3 "~" H 6075 1350 50  0001 C CNN
+	1    6075 1350
 	1    0    0    -1
 $EndComp
-Text Label 6950 1100 1    60   ~ 0
+Text Label 6075 1050 1    60   ~ 0
 5V
 Wire Wire Line
-	6950 1550 6950 1750
-Text Label 6950 1750 3    60   ~ 0
+	6075 1500 6075 1700
+Text Label 6075 1700 3    60   ~ 0
 GND
 Wire Wire Line
-	6950 1100 6950 1250
+	6075 1050 6075 1200
 $Comp
 L Connector_Generic:Conn_01x02 P17
@@
 	500  9600 10700 9600
 Wire Notes Line
-	10700 500  10700 17500
-Wire Notes Line
 	10700 7000 29500 7000
 Wire Notes Line
@@
 Wire Notes Line
 	500  12500 10700 12500
-Text Notes 7075 2125 0    60   ~ 0
+Text Notes 6200 2075 0    60   ~ 0
 power decoupling
 Text Notes 600  4200 0    100  ~ 0
@@
 Text Notes 600  12700 0    100  ~ 0
 Electrode Connection Subsystem
-Text Notes 10800 700  0    100  ~ 0
-Transimpedance Subsystem
 Text Notes 10800 7200 0    100  ~ 0
 Control & Reference Subsystem
@@
 Text Notes 21300 4325 0    50   ~ 10
 8. Replace R33, R34, R36  with 10k resistors\nDONE
+Wire Notes Line
+	8600 500  8600 4000
+Text Notes 10800 700  0    100  ~ 0
+Transimpedance Subsystem
+Wire Notes Line
+	10700 500  10700 17500
+Text Notes 9125 950  0    100  ~ 0
+Dummy headers \nfor auto assembly
+$Comp
+L dummy:header_14_pos UA2
+U 1 1 66C1CFA4
+P 9675 1650
+F 0 "UA2" H 9675 1840 50  0000 C CNN
+F 1 "header_14_pos" H 9675 1749 50  0000 C CNN
+F 2 "dummy:header_14_pos" H 9675 1575 50  0001 C CNN
+F 3 "" H 9675 1575 50  0001 C CNN
+	1    9675 1650
+	1    0    0    -1
+$EndComp
+$Comp
+L dummy:header_14_pos UB2
+U 1 1 66C1E55B
+P 9675 2050
+F 0 "UB2" H 9675 2240 50  0000 C CNN
+F 1 "header_14_pos" H 9675 2149 50  0000 C CNN
+F 2 "dummy:header_14_pos" H 9675 1975 50  0001 C CNN
+F 3 "" H 9675 1975 50  0001 C CNN
+	1    9675 2050
+	1    0    0    -1
+$EndComp
+$Comp
+L dummy:header_5_pos UC2
+U 1 1 66C1F9DF
+P 9675 2450
+F 0 "UC2" H 9675 2640 50  0000 C CNN
+F 1 "header_5_pos" H 9675 2549 50  0000 C CNN
+F 2 "dummy:header_5_pos" H 9675 2375 50  0001 C CNN
+F 3 "" H 9675 2375 50  0001 C CNN
+	1    9675 2450
+	1    0    0    -1
+$EndComp
 $EndSCHEMATC
